File: kicad/1mb mapper nms8280.kicad_sch (KiCad schematic)
At the start: 12 parts, among them IC147 74LS157, IC147B 74LS157, IC149 74LS670, IC149B 74LS670, J1 Conn_01x08_Pin

Commit message: Update KiCad design files from archive
Parts:
- renumbered CONN147 to CONN3, IC131B to IC131B1, IC147B to IC147B1, IC149B to IC149B1, IC157B to IC157B1, IC180B to IC180B1, IC147 to IC3
Connections:
- net GND: now also IC149B1.2 (D3), IC149B1.3 (D4)
- net Vcc: no longer CONN3.16 (Vcc)
Other:
- title: (none) -> Mapper 1MB MSX NMS8280
Changed lines of the file:
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@@
 	(generator_version "10.0")
 	(paper "A4")
+	(title_block
+		(title "Mapper 1MB MSX NMS8280")
+		(date "2026-08-30")
+	)
 	(text "To IC176 P11"
 		(exclude_from_sim no)
@@
 	)
 	(junction
+		(at 99.06 130.81)
+		(diameter 0)
+		(color 0 0 0 0)
+	)
+	(junction
 		(at 88.9 91.44)
 		(diameter 0)
@@
 	)
 	(junction
-		(at 97.79 116.84)
+		(at 96.52 114.3)
 		(diameter 0)
 		(color 0 0 0 0)
 	)
 	(junction
-		(at 95.25 130.81)
+		(at 144.78 114.3)
 		(diameter 0)
 		(color 0 0 0 0)
 	)
 	(junction
-		(at 92.71 114.3)
+		(at 88.9 99.06)
 		(diameter 0)
 		(color 0 0 0 0)
 	)
 	(junction
-		(at 144.78 114.3)
+		(at 101.6 116.84)
 		(diameter 0)
 		(color 0 0 0 0)
 	)
 	(junction
-		(at 88.9 99.06)
+		(at 104.14 133.35)
 		(diameter 0)
 		(color 0 0 0 0)
@@
 	)
 	(junction
-		(at 100.33 133.35)
+		(at 149.86 109.22)
 		(diameter 0)
 		(color 0 0 0 0)
 	)
 	(junction
-		(at 149.86 109.22)
+		(at 88.9 148.59)
 		(diameter 0)
 		(color 0 0 0 0)
 	)
 	(junction
-		(at 88.9 148.59)
+		(at 72.39 88.9)
 		(diameter 0)
 		(color 0 0 0 0)
 	)
 	(junction
-		(at 72.39 88.9)
+		(at 137.16 111.76)
 		(diameter 0)
 		(color 0 0 0 0)
@@
 	(wire
 		(pts
-			(xy 92.71 31.75) (xy 195.58 31.75)
+			(xy 96.52 31.75) (xy 195.58 31.75)
 		)
 		(stroke
@@
 	(wire
 		(pts
-			(xy 97.79 116.84) (xy 111.76 116.84)
+			(xy 142.24 111.76) (xy 142.24 81.28)
 		)
 		(stroke
@@
 	(wire
 		(pts
-			(xy 97.79 29.21) (xy 195.58 29.21)
+			(xy 101.6 29.21) (xy 195.58 29.21)
 		)
 		(stroke
@@
 	(wire
 		(pts
-			(xy 100.33 153.67) (xy 100.33 133.35)
+			(xy 104.14 153.67) (xy 104.14 133.35)
 		)
 		(stroke
@@
 	(wire
 		(pts
+			(xy 99.06 130.81) (xy 142.24 130.81)
+		)
+		(stroke
+			(width 0)
+			(type default)
+		)
+	)
+	(wire
+		(pts
 			(xy 142.24 130.81) (xy 142.24 116.84)
 		)
@@
 	(wire
 		(pts
-			(xy 26.67 38.1) (xy 95.25 38.1)
+			(xy 26.67 38.1) (xy 99.06 38.1)
 		)
 		(stroke
@@
 	(wire
 		(pts
-			(xy 100.33 133.35) (xy 100.33 40.64)
+			(xy 104.14 133.35) (xy 104.14 40.64)
 		)
 		(stroke
@@
 	(wire
 		(pts
-			(xy 97.79 116.84) (xy 97.79 29.21)
+			(xy 101.6 116.84) (xy 101.6 29.21)
 		)
 		(stroke
@@
 	(wire
 		(pts
-			(xy 95.25 161.29) (xy 118.11 161.29)
+			(xy 99.06 161.29) (xy 118.11 161.29)
 		)
 		(stroke
@@
 	(wire
 		(pts
-			(xy 95.25 130.81) (xy 95.25 161.29)
+			(xy 99.06 130.81) (xy 99.06 161.29)
 		)
 		(stroke
@@
 	(wire
 		(pts
-			(xy 102.87 151.13) (xy 118.11 151.13)
+			(xy 106.68 151.13) (xy 118.11 151.13)
 		)
 		(stroke
@@
 	(wire
 		(pts
-			(xy 92.71 31.75) (xy 92.71 114.3)
+			(xy 96.52 31.75) (xy 96.52 114.3)
 		)
 		(stroke
@@
 	(wire
 		(pts
-			(xy 95.25 130.81) (xy 95.25 38.1)
+			(xy 99.06 130.81) (xy 99.06 38.1)
 		)
 		(stroke
@@
 	(wire
 		(pts
-			(xy 118.11 158.75) (xy 97.79 158.75)
+			(xy 118.11 158.75) (xy 101.6 158.75)
 		)
 		(stroke
@@
 	(wire
 		(pts
-			(xy 102.87 135.89) (xy 149.86 135.89)
+			(xy 106.68 135.89) (xy 149.86 135.89)
 		)
 		(stroke
@@
 	(wire
 		(pts
-			(xy 134.62 168.91) (xy 92.71 168.91)
+			(xy 134.62 168.91) (xy 96.52 168.91)
 		)
 		(stroke
@@
 	(wire
 		(pts
-			(xy 102.87 151.13) (xy 102.87 135.89)
+			(xy 137.16 111.76) (xy 142.24 111.76)
+		)
+		(stroke
+			(width 0)
+			(type default)
+		)
+	)
+	(wire
+		(pts
+			(xy 106.68 151.13) (xy 106.68 135.89)
 		)
 		(stroke
@@
 	(wire
 		(pts
-			(xy 97.79 158.75) (xy 97.79 116.84)
+			(xy 101.6 158.75) (xy 101.6 116.84)
 		)
 		(stroke
@@
 	(wire
 		(pts
-			(xy 26.67 40.64) (xy 100.33 40.64)
+			(xy 26.67 40.64) (xy 104.14 40.64)
 		)
 		(stroke
@@
 	(wire
 		(pts
-			(xy 100.33 133.35) (xy 182.88 133.35)
+			(xy 137.16 109.22) (xy 137.16 111.76)
 		)
 		(stroke
@@
 	(wire
 		(pts
-			(xy 92.71 114.3) (xy 111.76 114.3)
+			(xy 104.14 133.35) (xy 182.88 133.35)
 		)
 		(stroke
@@
 	(wire
 		(pts
+			(xy 101.6 116.84) (xy 111.76 116.84)
+		)
+		(stroke
+			(width 0)
+			(type default)
+		)
+	)
+	(wire
+		(pts
 			(xy 76.2 146.05) (xy 76.2 140.97)
 		)
@@
 	(wire
 		(pts
-			(xy 118.11 153.67) (xy 100.33 153.67)
+			(xy 118.11 153.67) (xy 104.14 153.67)
 		)
 		(stroke
@@
 	(wire
 		(pts
+			(xy 124.46 81.28) (xy 142.24 81.28)
+		)
+		(stroke
+			(width 0)
+			(type default)
+		)
+	)
+	(wire
+		(pts
 			(xy 17.78 21.59) (xy 17.78 168.91)
 		)
@@
 	(wire
 		(pts
-			(xy 64.77 50.8) (xy 64.77 156.21)
+			(xy 96.52 114.3) (xy 111.76 114.3)
 		)
 		(stroke
@@
 	(wire
 		(pts
-			(xy 130.81 161.29) (xy 134.62 161.29)
+			(xy 64.77 50.8) (xy 64.77 156.21)
 		)
 		(stroke
@@
 	(wire
 		(pts
-			(xy 195.58 36.83) (xy 195.58 39.37)
+			(xy 130.81 161.29) (xy 134.62 161.29)
 		)
 		(stroke
@@
 	(wire
 		(pts
-			(xy 88.9 99.06) (xy 88.9 101.6)
+			(xy 195.58 36.83) (xy 195.58 39.37)
 		)
 		(stroke
@@
 	(wire
 		(pts
-			(xy 92.71 168.91) (xy 92.71 114.3)
+			(xy 88.9 99.06) (xy 88.9 101.6)
 		)
 		(stroke
@@
 	(wire
 		(pts
-			(xy 74.93 158.75) (xy 76.2 158.75)
+			(xy 96.52 168.91) (xy 96.52 114.3)
 		)
 		(stroke
@@
 	(wire
 		(pts
-			(xy 72.39 88.9) (xy 76.2 88.9)
+			(xy 74.93 158.75) (xy 76.2 158.75)
 		)
 		(stroke
@@
 	(wire
 		(pts
-			(xy 95.25 130.81) (xy 142.24 130.81)
+			(xy 72.39 88.9) (xy 76.2 88.9)
 		)
 		(stroke
@@
 		)
 	)
-	(label "Vcc"
-		(at 276.86 27.94 0)
-		(effects
-			(font
-				(size 0.508 0.508)
-			)
-			(justify left bottom)
-		)
-	)
 	(label "IC131_P1_IC131B"
 		(at 118.11 148.59 180)
@@
 		(in_pos_files yes)
 		(dnp no)
-		(property "Reference" "IC180B"
+		(property "Reference" "IC180B1"
 			(at 91.694 139.192 0)
 			(show_name no)
@@
 			(project "1mb mapper nms8280"
 				(path "/f3c5738e-f967-4261-9d5d-47df8254fb38"
-					(reference "IC180B")
+					(reference "IC180B1")
 					(unit 1)
 				)
@@
 		(in_pos_files yes)
 		(dnp no)
-		(property "Reference" "IC149B"
+		(property "Reference" "IC149B1"
 			(at 127.508 80.772 0)
 			(show_name no)
@@
 			(project "1mb mapper nms8280"
 				(path "/f3c5738e-f967-4261-9d5d-47df8254fb38"
-					(reference "IC149B")
+					(reference "IC149B1")
 					(unit 1)
 				)
@@
 		(in_pos_files yes)
 		(dnp no)
-		(property "Reference" "IC131B"
+		(property "Reference" "IC131B1"
 			(at 126.7139 142.24 0)
 			(show_name no)
@@
 			(project "1mb mapper nms8280"
 				(path "/f3c5738e-f967-4261-9d5d-47df8254fb38"
-					(reference "IC131B")
+					(reference "IC131B1")
 					(unit 1)
 				)
@@
 		(dnp no)
 		(fields_autoplaced yes)
-		(property "Reference" "IC147"
+		(property "Reference" "IC3"
 			(at 244.7133 13.97 0)
 			(show_name no)
@@
 			(project "1mb mapper nms8280"
 				(path "/f3c5738e-f967-4261-9d5d-47df8254fb38"
-					(reference "IC147")
+					(reference "IC3")
 					(unit 1)
 				)
@@
 		(in_pos_files yes)
 		(dnp no)
-		(property "Reference" "IC157B"
+		(property "Reference" "IC157B1"
 			(at 91.44 82.55 0)
 			(show_name no)
@@
 			(project "1mb mapper nms8280"
 				(path "/f3c5738e-f967-4261-9d5d-47df8254fb38"
-					(reference "IC157B")
+					(reference "IC157B1")
 					(unit 1)
 				)
@@
 		(in_pos_files yes)
 		(dnp no)
-		(property "Reference" "CONN147"
+		(property "Reference" "CONN3"
 			(at 277.622 20.574 0)
 			(show_name no)
@@
 			(project "1mb mapper nms8280"
 				(path "/f3c5738e-f967-4261-9d5d-47df8254fb38"
-					(reference "CONN147")
+					(reference "CONN3")
 					(unit 1)
 				)
@@
 		(dnp no)
 		(fields_autoplaced yes)
-		(property "Reference" "IC147B"
+		(property "Reference" "IC147B1"
 			(at 210.4233 13.97 0)
 			(show_name no)
@@
 			(project "1mb mapper nms8280"
 				(path "/f3c5738e-f967-4261-9d5d-47df8254fb38"
-					(reference "IC147B")
+					(reference "IC147B1")
 					(unit 1)
 				)

Commit message: Update KiCad project from local archive
Parts:
- IC147: renamed from IC3; footprint (none) -> Package_SO:SOIC-16W_5.3x10.2mm_P1.27mm
- IC147B1: footprint (none) -> Package_SO:SOIC-16W_5.3x10.2mm_P1.27mm
- J1: footprint (none) -> Connector_PinHeader_2.54mm:PinHeader_1x08_P2.54mm_Horizontal
- renumbered CONN3 to CONN147
Connections:
- net A8_IC147B_P4: now reaches IC147B1.4 (Za)
- net A9_IC147B_P7: now reaches IC147B1.7 (Zb)
Changed lines of the file:
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@@
+		)
+	)
+	(global_label "A9_IC147B_P7"
+		(shape input)
+		(at 220.98 29.21 0)
+		(fields_autoplaced yes)
+		(effects
+			(font
+				(size 0.508 0.508)
+			)
+			(justify left)
+		)
+		(property "Intersheetrefs" "${INTERSHEET_REFS}"
+			(at 237.4513 29.21 0)
+			(hide yes)
+			(show_name no)
+			(do_not_autoplace no)
+			(effects
+				(font
+					(size 1.27 1.27)
+				)
+				(justify left)
+			)
+		)
+	)
+	(global_label "A8_IC147B_P4"
+		(shape input)
+		(at 220.98 21.59 0)
+		(fields_autoplaced yes)
+		(effects
+			(font
+				(size 0.508 0.508)
+			)
+			(justify left)
+		)
+		(property "Intersheetrefs" "${INTERSHEET_REFS}"
+			(at 237.4513 21.59 0)
+			(hide yes)
+			(show_name no)
+			(do_not_autoplace no)
+			(effects
+				(font
+					(size 1.27 1.27)
+				)
+				(justify left)
+			)
 		)
 	)
@@
 		(dnp no)
 		(fields_autoplaced yes)
-		(property "Reference" "IC3"
+		(property "Reference" "IC147"
 			(at 244.7133 13.97 0)
 			(show_name no)
@@
 			)
 		)
-		(property "Footprint" ""
+		(property "Footprint" "Package_SO:SOIC-16W_5.3x10.2mm_P1.27mm"
 			(at 242.57 36.83 0)
 			(hide yes)
@@
 			(project "1mb mapper nms8280"
 				(path "/f3c5738e-f967-4261-9d5d-47df8254fb38"
-					(reference "IC3")
+					(reference "IC147")
 					(unit 1)
 				)
@@
 			)
 		)
-		(property "Footprint" ""
+		(property "Footprint" "Connector_PinHeader_2.54mm:PinHeader_1x08_P2.54mm_Horizontal"
 			(at 21.59 40.64 0)
 			(hide yes)
@@
 		(in_pos_files yes)
 		(dnp no)
-		(property "Reference" "CONN3"
+		(property "Reference" "CONN147"
 			(at 277.622 20.574 0)
 			(show_name no)
@@
 			(project "1mb mapper nms8280"
 				(path "/f3c5738e-f967-4261-9d5d-47df8254fb38"
-					(reference "CONN3")
+					(reference "CONN147")
 					(unit 1)
 				)
@@
 			)
 		)
-		(property "Footprint" ""
+		(property "Footprint" "Package_SO:SOIC-16W_5.3x10.2mm_P1.27mm"
 			(at 208.28 36.83 0)
 			(hide yes)
